Commit message: Removed parent joint from tracker macro.

File: xacro/tracker.xacro (robot description, xacro)
@@ -74,10 +74,6 @@
   </xacro:macro>
   <!-- INTEL REALSENSE T265 -->
-  <xacro:macro name="realsense_T265" params="sensor_name parent_link rate *origin">
-    <joint name="${sensor_name}_odom_frame_joint" type="fixed">
-        <parent link="${parent_link}"/>
-        <child link="${sensor_name}_odom_frame"/>
-        <xacro:insert_block name="origin"/>
-    </joint>
+  <xacro:macro name="realsense_T265" params="sensor_name rate *origin">
+    <!-- Removed joint to parent link. Add externally. -->
     <joint name="${sensor_name}_pose_frame_joint" type="fixed">
         <parent link="${sensor_name}_odom_frame"/>

Commit message: Tweaking t265 links a bit more

File: xacro/tracker.xacro (robot description, xacro)
@@ -76,11 +76,11 @@
   <xacro:macro name="realsense_T265" params="sensor_name rate *origin">
     <!-- Removed joint to parent link. Add externally. -->
-    <joint name="${sensor_name}_pose_frame_joint" type="fixed">
-        <parent link="${sensor_name}_odom_frame"/>
-        <child link="${sensor_name}_pose_frame"/>
-        <origin rpy="0 0 0" xyz="0 0 0"/> <!-- check on real hw -->
+    <link name="${sensor_name}_pose_frame"/>
+    <joint name="${sensor_name}_pose_joint" type="fixed">
+        <origin rpy="0 0 0" xyz="0 0 0"/>
+        <parent link="${sensor_name}_pose_frame"/>
+        <child link="${sensor_name}_link"/>
     </joint>
-    <link name="${sensor_name}_odom_frame"/>
-    <link name="${sensor_name}_pose_frame">
+    <link name="${sensor_name}_link">
         <visual>
             <origin rpy="1.57 0 1.57" xyz="0 0 0"/>
@@ -105,10 +105,4 @@
         </inertial>
     </link>
-    <joint name="${sensor_name}_joint" type="fixed">
-        <parent link="${sensor_name}_pose_frame"/>
-        <child link="${sensor_name}_link"/>
-        <origin rpy="0 0 0" xyz="0 0 0"/> <!-- check on real hw -->
-    </joint>
-    <link name="${sensor_name}_link"/>
     <joint name="${sensor_name}_fisheye1_joint" type="fixed">
         <parent link="${sensor_name}_link"/>
@@ -161,5 +155,5 @@
             <plugin filename="libgazebo_ros_imu_sensor.so" name="imu_plugin">
                 <topicName>${sensor_name}/gyro/sample</topicName>
-                <bodyName>${sensor_name}_pose_frame</bodyName>
+                <bodyName>${sensor_name}_link</bodyName>
                 <updateRateHZ>${rate}</updateRateHZ>
                 <gaussianNoise>0.000001</gaussianNoise>
@@ -180,5 +174,5 @@
             <alwaysOn>true</alwaysOn>
             <updateRate>${rate}</updateRate>
-            <bodyName>${sensor_name}_odom_frame</bodyName>
+            <bodyName>${sensor_name}_pose_frame</bodyName>
             <topicName>${sensor_name}/odom/sample</topicName>
             <gaussianNoise>0.001</gaussianNoise>

Commit message: Removed pose link from tracker.xacro

File: xacro/tracker.xacro (robot description, xacro)
@@ -74,12 +74,6 @@
   </xacro:macro>
   <!-- INTEL REALSENSE T265 -->
-  <xacro:macro name="realsense_T265" params="sensor_name rate *origin">
+  <xacro:macro name="realsense_T265" params="sensor_name rate">
     <!-- Removed joint to parent link. Add externally. -->
-    <link name="${sensor_name}_pose_frame"/>
-    <joint name="${sensor_name}_pose_joint" type="fixed">
-        <origin rpy="0 0 0" xyz="0 0 0"/>
-        <parent link="${sensor_name}_pose_frame"/>
-        <child link="${sensor_name}_link"/>
-    </joint>
     <link name="${sensor_name}_link">
         <visual>
@@ -174,5 +168,5 @@
             <alwaysOn>true</alwaysOn>
             <updateRate>${rate}</updateRate>
-            <bodyName>${sensor_name}_pose_frame</bodyName>
+            <bodyName>${sensor_name}_link</bodyName>
             <topicName>${sensor_name}/odom/sample</topicName>
             <gaussianNoise>0.001</gaussianNoise>

Commit message: Tweaking t265 more

File: xacro/tracker.xacro (robot description, xacro)
@@ -76,4 +76,10 @@
   <xacro:macro name="realsense_T265" params="sensor_name rate">
     <!-- Removed joint to parent link. Add externally. -->
+    <link name="${sensor_name}_pose_frame"/>
+    <joint name="${sensor_name}_pose_joint" type="fixed">
+        <origin rpy="0 0 0" xyz="0 0 0"/>
+        <parent link="${sensor_name}_pose_frame"/>
+        <child link="${sensor_name}_link"/>
+    </joint>
     <link name="${sensor_name}_link">
         <visual>
@@ -164,9 +170,14 @@
     </joint>
     <link name="${sensor_name}_accel_frame"/> <!-- dummy -->
-    <gazebo> <!-- odometry -->
+    <!-- For simplicity, just publishes odometry for base_link
+    Otherwise, the t265_pose_link has to become the base link -->
+    <!-- Also, need to set frameName to world, since the plugin
+    complains if the frame doesn't exist. However, this is
+    renamed to odom when publishing tf -->
+    <gazebo>
         <plugin name="p3d_base_controller" filename="libgazebo_ros_p3d.so">
             <alwaysOn>true</alwaysOn>
             <updateRate>${rate}</updateRate>
-            <bodyName>${sensor_name}_link</bodyName>
+            <bodyName>base_link</bodyName>
             <topicName>${sensor_name}/odom/sample</topicName>
             <gaussianNoise>0.001</gaussianNoise>
